File: Verzerrer.brd (EAGLE design)
At the start: 100 x 80 mm, 17 parts, among them IC1 LM741P

Commit message: Board bearbeitet
Parts:
- moved R3 72.7 mm to (80.0, 30.5)
- moved C1 47.6 mm to (8.89, 73.7)
- moved LSP1 35.8 mm to (19.1, 31.8)
- moved R1 8.13 mm to (6.35, 31.8), turned to 90 degrees
- moved R2 6.48 mm to (40.6, 31.8), turned to 270 degrees
- moved R6 5.08 mm to (7.62, 47.0)
- moved D2 5.08 mm to (49.5, 53.3), turned to 90 degrees
- turned D1 to 90 degrees
Routing:
- net N$7: track 0.00 -> 290.1 mm
- net N$3: track 0.00 -> 95.7 mm
- net N$6: track 0.00 -> 92.5 mm
- net N$1: track 0.00 -> 84.0 mm
- net N$9: track 0.00 -> 61.3 mm
- net N$4: track 0.00 -> 35.7 mm
- net N$2: track 0.00 -> 30.4 mm
- net N$5: track 0.00 -> 23.7 mm
- net N$10: track 0.00 -> 19.6 mm
- net N$8: track 0.00 -> 15.2 mm
